File: PCB-DNS-DriveBy/DNS-DriveBy/DNS-DriveBy.kicad_sch (KiCad schematic)
At the start: 20 parts, among them J1 JST 2.0, J2 Conn_01x04, J3 Conn_01x03, J4 Micro_SD_Card_Det, Q1 2N3904, Q2 2N3904, SW1 SW_SPST, U1 D1 Mini, U2 NEO-6M

Commit message: publish v1.3 design files
Parts:
- added R3: 10K, Resistor_THT:R_Axial_DIN0207_L6.3mm_D2.5mm_P7.62mm_Horizontal, symbol Device:R_Small_US
- J2: value Conn_01x04 -> SH1106
- J4: footprint (none) -> DNS-DriveBy:MicroSD
Connections:
- net +3V3: now also J2.1 (Pin_1); no longer J2.2 (Pin_2)
- net +BATT: now also J1.1 (Pin_1), U2.1 (VCC); no longer J1.2 (Pin_2), JP1.1 (A), Q2.3 (C)
- net GND: now also J2.2 (Pin_2), J4.11 (SHIELD), JP1.1 (A), Q2.1 (E), R3.2; no longer J2.1 (Pin_1), U2.4 (GND)
- net SS: now also R3.1
- net at JP5.2 (B), SW1.2 (B): now also J1.2 (Pin_2); no longer J1.1 (Pin_1)
- net at JP1.2 (C): now also U2.4 (GND); no longer U2.1 (VCC)
- net at JP1.3 (B): now also Q2.3 (C); no longer Q2.1 (E)
Other:
- moved on the sheet: J1, J2, JP1, JP2, JP3, JP4, JP5, Q2, R4, R5, R6, SW1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
